Commit message: Fix the URDF posture of the car, adjust the configuration of fake_joint_states and rviz

File: src/mbot_description/urdf/macros_common.xacro (robot description, xacro)
@@ -6,7 +6,9 @@
     <inertial>
       <mass value="${mass}"/>
-      <inertia ixx="${0.5 * mass * radius * radius}" ixy="0" ixz="0"
-               iyy="${mass * (3 * radius * radius + length * length) / 12}" iyz="0"
-               izz="${mass * (3 * radius * radius + length * length) / 12}"/>
+      <inertia ixx="${mass * (3 * radius * radius + length * length) / 12}"
+              ixy="0" ixz="0"
+              iyy="${mass * (3 * radius * radius + length * length) / 12}"
+              iyz="0"
+              izz="${0.5 * mass * radius * radius}"/>
     </inertial>
   </xacro:macro>

File: src/mbot_description/urdf/mbot.xacro (robot description, xacro)
@@ -79,4 +79,5 @@
           <cylinder radius="${wheel_radius}" length="${wheel_width}"/>
         </geometry>
+        <!-- URDF cylinder 的 length 沿局部 Z 轴；绕 X 转 90° 使长轴沿 Y，盘面朝前后。 -->
         <origin xyz="0 0 0" rpy="${pi/2} 0 0"/>
         <material name="black"/>
